File: robokon2026_sub.kicad_sch (KiCad schematic)
At the start: 15 parts, among them J1 Conn_01x02_Socket, J2 12402054M611A, J3 Conn_01x05_Pin, U1 NUCLEO-F303K8, U2 ATA6561-GAQW-N, U4 AZ1117CH2-5.0, U5 LD1117S50TR_SOT223

Commit message: add robokon2026_sub/pcb
Parts:
- C1, C2, C3, C4, C5, C6: footprint (none) -> Capacitor_THT:CP_Radial_D6.3mm_P2.50mm
- D1: footprint (none) -> Diode_SMD:D_SMC
- R1: footprint Resistor_SMD:R_0508_1220Metric_Pad1.12x2.15mm_HandSolder -> Resistor_SMD:R_0603_1608Metric_Pad0.98x0.95mm_HandSolder
Connections:
- net A renamed Phase_A
- net B renamed Phase_B
- net X renamed Phase_X
Changed lines of the file:
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@@
 		)
 	)
-	(label "X"
+	(label "Phase_X"
 		(at 104.14 142.24 0)
 		(effects
@@
 		)
 	)
-	(label "B"
+	(label "Phase_B"
 		(at 55.88 72.39 270)
 		(effects
@@
 		)
 	)
-	(label "X"
+	(label "Phase_X"
 		(at 63.5 72.39 270)
 		(effects
@@
 		)
 	)
-	(label "A"
+	(label "Phase_A"
 		(at 60.96 72.39 270)
 		(effects
@@
 		)
 	)
-	(label "A"
+	(label "Phase_A"
 		(at 104.14 127 0)
 		(effects
@@
 		)
 	)
-	(label "B"
+	(label "Phase_B"
 		(at 104.14 129.54 0)
 		(effects
@@
 			)
 		)
-		(property "Footprint" ""
+		(property "Footprint" "Capacitor_THT:CP_Radial_D6.3mm_P2.50mm"
 			(at 117.8052 135.89 0)
 			(effects
@@
 			)
 		)
-		(property "Footprint" ""
+		(property "Footprint" "Capacitor_THT:CP_Radial_D6.3mm_P2.50mm"
 			(at 108.9152 105.41 0)
 			(effects
@@
 			)
 		)
-		(property "Footprint" ""
+		(property "Footprint" "Capacitor_THT:CP_Radial_D6.3mm_P2.50mm"
 			(at 177.4952 46.99 0)
 			(effects
@@
 			)
 		)
-		(property "Footprint" ""
+		(property "Footprint" "Capacitor_THT:CP_Radial_D6.3mm_P2.50mm"
 			(at 125.4252 46.99 0)
 			(effects
@@
 			)
 		)
-		(property "Footprint" "Resistor_SMD:R_0508_1220Metric_Pad1.12x2.15mm_HandSolder"
+		(property "Footprint" "Resistor_SMD:R_0603_1608Metric_Pad0.98x0.95mm_HandSolder"
 			(at 176.022 135.89 90)
 			(effects
@@
 			)
 		)
-		(property "Footprint" ""
+		(property "Footprint" "Capacitor_THT:CP_Radial_D6.3mm_P2.50mm"
 			(at 149.5552 46.99 0)
 			(effects
@@
 			)
 		)
-		(property "Footprint" ""
+		(property "Footprint" "Capacitor_THT:CP_Radial_D6.3mm_P2.50mm"
 			(at 100.0252 46.99 0)
 			(effects
@@
 			)
 		)
-		(property "Footprint" ""
+		(property "Footprint" "Diode_SMD:D_SMC"
 			(at 62.23 31.75 0)
 			(effects

Commit message: improvement1/robokon2026_sub
Parts:
- removed D1: D_Schottky, Diode_SMD:D_SMC, symbol Device:D_Schottky
- removed U2: ATA6561-GAQW-N, footprints:SOIC8_4P9X3P9MC_MCH, symbol ATA6561_GAQW_N:ATA6561-GAQW-N
- added D2: D_Schottky, Diode_SMD:D_SMC, symbol Device:D_Schottky
- added J4: Conn_01x02_Pin, Connector_AMASS:AMASS_XT30PW-M_1x02_P2.50mm_Horizontal, symbol Connector:Conn_01x02_Pin
- added J5: 12402054M611A, 12402054M611A:AMPHENOL_12402054M611A, symbol 12402054M611A:12402054M611A
- added U2: ATA6561-GAQW-N, ATA6561_GAQW_N:SOIC8_4P9X3P9MC_MCH, symbol ATA6561-GAQW-N:ATA6561-GAQW-N
- C1, C3, C4, C5, C6: footprint Capacitor_THT:CP_Radial_D6.3mm_P2.50mm -> Capacitor_SMD:C_0805_2012Metric_Pad1.18x1.45mm_HandSolder
- C2: footprint Capacitor_THT:CP_Radial_D6.3mm_P2.50mm -> Capacitor_THT:CP_Radial_D10.0mm_P5.00mm
- J3: footprint Connector_PinHeader_2.54mm:PinHeader_1x05_P2.54mm_Vertical -> Connector_JST:JST_XH_S5B-XH-A_1x05_P2.50mm_Horizontal
Connections:
- net +12V: now also J1.2 (Pin_2), D2.2 (A), J4.1 (Pin_1)
- net +3V3: now also U2.5 (VIO)
- net +5V: now also U2.3 (VCC)
- net CAN_H: now also J5.A6 (D1+), J5.B6 (D2+), U2.7 (CANH)
- net CAN_L: now also J5.A7 (D1-), J5.B7 (D2-), U2.6 (CANL)
- net CAN_RX: now also U2.4 (RXD)
- net CAN_TX: now also U2.1 (TXD)
- net GND: now also D2.1 (K), J4.2 (Pin_2), J5.A1 (GND_A), J5.A12 (GND_A__1), J5.B1 (GND_B), J5.B12 (GND_B__1), J5.S1 (SHIELD), J5.S2 (SHIELD__1), J5.S3 (SHIELD__2), J5.S4 (SHIELD__3), U2.2 (GND), U2.8 (STBY)
- no-connect marks 28 -> 34
Other:
- moved on the sheet: J1

Commit message: improvement2/robokon2026_sub
Parts:
- removed U4: AZ1117CH2-5.0, Package_TO_SOT_SMD:SOT-223-3_TabPin2, symbol Regulator_Linear:AZ1117CH2-5.0
- removed U5: LD1117S50TR_SOT223, Package_TO_SOT_SMD:SOT-223-3_TabPin2, symbol Regulator_Linear:LD1117S50TR_SOT223
- added U4: AZ1117CH2-3.3, Package_TO_SOT_SMD:SOT-223-3_TabPin2, symbol Regulator_Linear:AZ1117CH2-3.3
- added U6: LD1117S50TR_SOT223, Package_TO_SOT_SMD:SOT-223-3_TabPin2, symbol Regulator_Linear:LD1117S50TR_SOT223
Connections:
- net +12V: now also C5.1, U6.3 (VI); no longer C3.1
- net +3V3: now also C4.1, U4.3 (OUT); no longer C6.1
- net +5V: now also C3.1, C6.1, U4.1 (IN), U6.2 (VO); no longer C4.1, C5.1
- net GND: now also U4.2 (GND), U6.1 (GND)
Other:
- moved on the sheet: C3, C4, C5, C6
