File: robokon2026_sub.kicad_pcb (KiCad board)
At the start: 2 copper layers, 80 x 50 mm, 19 parts, among them J1 Conn_01x02_Socket, J2 12402054M611A, J3 Conn_01x05_Pin, U1 NUCLEO-F303K8, U2 ATA6561-GAQW-N, U4 AZ1117CH2-5.0, U5 LD1117S50TR_SOT223

Commit message: improvement1/robokon2026_sub
Parts:
- removed D1: D_Schottky, Diode_SMD:D_SMC
- added D2: D_Schottky, Diode_SMD:D_SMC, F.Cu at (144.0, 97.4)
- added J4: Conn_01x02_Pin, Connector_AMASS:AMASS_XT30PW-M_1x02_P2.50mm_Horizontal, F.Cu at (136.3, 81.2)
- added J5: 12402054M611A, 12402054M611A:AMPHENOL_12402054M611A, F.Cu at (128.9, 69.3)
- C1, C3, C4, C5, C6: footprint Capacitor_THT:CP_Radial_D6.3mm_P2.50mm -> Capacitor_SMD:C_0805_2012Metric_Pad1.18x1.45mm_HandSolder
- C2: footprint Capacitor_THT:CP_Radial_D6.3mm_P2.50mm -> Capacitor_THT:CP_Radial_D10.0mm_P5.00mm
- J3: footprint Connector_PinHeader_2.54mm:PinHeader_1x05_P2.54mm_Vertical -> Connector_JST:JST_XH_S5B-XH-A_1x05_P2.50mm_Horizontal
- U2: footprint footprints:SOIC8_4P9X3P9MC_MCH -> ATA6561_GAQW_N:SOIC8_4P9X3P9MC_MCH
- moved J3 64.7 mm to (184.7, 95.6), turned to 90 degrees
- moved C6 11.3 mm to (170.8, 100.1)
- moved J2 11.1 mm to (128.9, 74.3)
- moved C2 8.33 mm to (176.5, 89.2)
- moved C5 8.16 mm to (165.4, 100.0)
- moved R1 7.51 mm to (151.0, 84.5)
- moved U2 7.31 mm to (156.2, 84.4)
- moved U5 6.90 mm to (166.6, 92.4)
- moved C1 6.51 mm to (158.5, 100.2), turned to -90 degrees
- moved J1 1.95 mm to (136.2, 100.5)
- moved C3 1.90 mm to (152.2, 100.2)
- moved C4 1.61 mm to (161.6, 100.2)
- moved U1 0.68 mm to (167.0, 70.7)
Connections:
- J1 pad 2: Net-(D1-K) -> +12V
Routing:
- net /Phase_X: track 46.8 -> 25.1 mm, vias 1 -> 2
- net +5V: track 56.1 -> 37.8 mm, vias 2 -> 1
- net /CAN_L: track 46.0 -> 64.1 mm
- net GND: track 18.9 -> 1.93 mm, vias 117 -> 167
- net +12V: track 6.31 -> 16.4 mm
- net Net-(D1-K): track 9.00 -> 0.00 mm
- net /Phase_B: track 34.7 -> 28.4 mm, vias 0 -> 1
- net /CAN_RX: track 25.6 -> 21.1 mm
- net +3V3: track 52.4 -> 56.8 mm, vias 1 -> 4
- net /CAN_TX: track 29.3 -> 31.7 mm, vias 1 -> 2
- net /CAN_H: track 32.4 -> 33.8 mm
- net /Phase_A: track 33.0 -> 33.8 mm, vias 0 -> 1
Other:
- board text added: "Phase_B"
- board text removed: "Phase_C"

Commit message: improvement2/robokon2026_sub
Parts:
- removed U5: LD1117S50TR_SOT223, Package_TO_SOT_SMD:SOT-223-3_TabPin2
- added U6: LD1117S50TR_SOT223, Package_TO_SOT_SMD:SOT-223-3_TabPin2, F.Cu at (152.5, 93.2)
- U4: value AZ1117CH2-5.0 -> AZ1117CH2-3.3
- moved C5 13.4 mm to (152.0, 100.5)
- moved C3 12.8 mm to (165.0, 100.2)
- moved C4 9.40 mm to (171.0, 100.2)
- moved C6 9.15 mm to (161.6, 100.2)
- moved U4 6.52 mm to (161.0, 93.0)
Connections:
- C3 pad 1: +12V -> +5V
- C4 pad 1: +5V -> +3V3
- C5 pad 1: +5V -> +12V
- C6 pad 1: +3V3 -> +5V
- U4 pad 1: +12V -> +5V
- U4 pad 3: +5V -> +3V3
Routing:
- net +5V: track 37.8 -> 51.4 mm
- net +12V: track 16.4 -> 20.7 mm
- net GND: vias 167 -> 164
